File: stmsplat1.kicad_pcb (KiCad board)
At the start: 2 copper layers, 14 parts, among them CN1 C_Pack04, CN10 Conn_01x34_Male, CN7 Conn_01x20_Male, CN8 Conn_01x16_Male, CN9 Conn_01x30_Male, J1 Conn_Coaxial, J2 Conn_Coaxial, J3 Conn_Coaxial, U1 NUCLEO144-F746ZG, U2 SA630D-RF_Switch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

Commit message: Added Arduino Header Labels
Connections:
- net Net-(CN10-Pad10) renamed /PE13
- net Net-(CN10-Pad11) renamed /PF4
- net Net-(CN10-Pad12) renamed /PF15
- net Net-(CN10-Pad13) renamed /PB6
- net Net-(CN10-Pad14) renamed /PG14
- net Net-(CN10-Pad15) renamed /PB2
- net Net-(CN10-Pad16) renamed /PG9
- net Net-(CN10-Pad18) renamed /PE8
- net Net-(CN10-Pad19) renamed /PD13
- net Net-(CN10-Pad2) renamed /PF13
- net Net-(CN10-Pad20) renamed /PE7
- net Net-(CN10-Pad21) renamed /PD12
- net Net-(CN10-Pad23) renamed /PD11
- net Net-(CN10-Pad24) renamed /PE10
- net Net-(CN10-Pad26) renamed /PE12
- net Net-(CN10-Pad28) renamed /PE14
- net Net-(CN10-Pad29) renamed /PA0
- net Net-(CN10-Pad3) renamed /AGND
- net Net-(CN10-Pad30) renamed /PE15
- net Net-(CN10-Pad31) renamed /PB0
- net Net-(CN10-Pad32) renamed /PB10
- net Net-(CN10-Pad33) renamed /PE0
- net Net-(CN10-Pad34) renamed /PB11
- net Net-(CN10-Pad4) renamed /PE9
- net Net-(CN10-Pad6) renamed /PE11
- net Net-(CN10-Pad7) renamed /PB1
- net Net-(CN10-Pad8) renamed /PF14
- net Net-(CN10-Pad9) renamed /PC2
- net Net-(CN7-Pad1) renamed /PC6
- net Net-(CN7-Pad10) renamed /PA5
- net Net-(CN7-Pad11) renamed /PC7
- net Net-(CN7-Pad12) renamed /PA6
- net Net-(CN7-Pad13) renamed /PB5
- net Net-(CN7-Pad15) renamed /PB3
- net Net-(CN7-Pad16) renamed /PD14
- net Net-(CN7-Pad17) renamed /PA4
- net Net-(CN7-Pad18) renamed /PD15
- net Net-(CN7-Pad19) renamed /PB4
- net Net-(CN7-Pad2) renamed /PB8
- net Net-(CN7-Pad20) renamed /PF12
- net Net-(CN7-Pad3) renamed /PB15
- net Net-(CN7-Pad4) renamed /PB9
- net Net-(CN7-Pad5) renamed /PB13
- net Net-(CN7-Pad7) renamed /PB12
- net Net-(CN7-Pad9) renamed /PA15
- net Net-(CN9-Pad1) renamed /PA3
- net Net-(CN9-Pad10) renamed /PD3
- net Net-(CN9-Pad11) renamed /PF10
- net Net-(CN9-Pad16) renamed /PE4
- net Net-(CN9-Pad17) renamed /PF2
- net Net-(CN9-Pad18) renamed /PE5
- net Net-(CN9-Pad19) renamed /PF1
- net Net-(CN9-Pad2) renamed /PD7
- net Net-(CN9-Pad20) renamed /PE6
- net Net-(CN9-Pad21) renamed /PF0
- net Net-(CN9-Pad22) renamed /PE3
- net Net-(CN9-Pad24) renamed /PF8
- net Net-(CN9-Pad25) renamed /PD0
- net Net-(CN9-Pad26) renamed /PF7
- net Net-(CN9-Pad27) renamed /PD1
- net Net-(CN9-Pad28) renamed /PF9
- net Net-(CN9-Pad29) renamed /PG0
- net Net-(CN9-Pad3) renamed /PC0
- net Net-(CN9-Pad30) renamed /PG1
- net Net-(CN9-Pad4) renamed /PD6
- net Net-(CN9-Pad5) renamed /PC3
- net Net-(CN9-Pad6) renamed /PD5
- net Net-(CN9-Pad7) renamed /PF3
- net Net-(CN9-Pad8) renamed /PD4
- net Net-(CN9-Pad9) renamed /PF5
- CN10 pad 1: Net-(CN10-Pad1) -> /AVDD
- CN10 pad 17: Net-(CN10-Pad17) -> /GND
- CN10 pad 22: Net-(CN10-Pad22) -> /GND
- CN10 pad 25: Net-(CN10-Pad25) -> /PE2
- CN10 pad 27: Net-(CN10-Pad27) -> /GND
- CN10 pad 5: Net-(CN10-Pad5) -> /GND
- CN7 pad 14: Net-(CN7-Pad14) -> /PA7
- CN7 pad 6: Net-(CN7-Pad6) -> /AVDD
- CN7 pad 8: Net-(CN7-Pad8) -> /GND
- CN9 pad 12: Net-(CN9-Pad12) -> /GND
- CN9 pad 14: Net-(CN9-Pad14) -> /PE2
- CN9 pad 15: Net-(CN9-Pad15) -> /PA7
- CN9 pad 23: Net-(CN9-Pad23) -> /GND
