File: stmsplat1.sch (KiCad schematic (older format))
At the start: 5 parts, among them CN10 Conn_01x34_Male, CN7 Conn_01x20_Male, CN8 Conn_01x16_Male, CN9 Conn_01x30_Male, U1 NUCLEO144-F746ZG

Commit message: Experimented with KiCad operations
Tried new symbols  / footprints etc
Parts:
- added CN?: C_Pack04, symbol c_pack04:C_Pack04
- added J1, J2, J3: Conn_Coaxial, Connector_Coaxial:SMB_Jack_Vertical, symbol Connector:Conn_Coaxial
- added RN1, RN2: R_Pack04, Resistor_SMD:R_Array_Convex_4x1206, symbol Device:R_Pack04
- added U2: SA630D, Package_SO:SOIC-8_3.9x4.9mm_P1.27mm, symbol RF_Switch:SA630D
Connections:
- wire segments 0 -> 9
Changed lines of the file:
@@
+	1    0    0    -1
+$EndComp
+$Comp
+L Connector:Conn_Coaxial J3
+U 1 1 5BD26EDD
+P 14250 1700
+F 0 "J3" H 14349 1676 50  0000 L CNN
+F 1 "Conn_Coaxial" H 14349 1585 50  0000 L CNN
+F 2 "Connector_Coaxial:SMB_Jack_Vertical" H 14250 1700 50  0001 C CNN
+F 3 " ~" H 14250 1700 50  0001 C CNN
+	1    14250 1700
+	1    0    0    -1
+$EndComp
+$Comp
+L Connector:Conn_Coaxial J2
+U 1 1 5BD2707C
+P 14150 2550
+F 0 "J2" H 14249 2526 50  0000 L CNN
+F 1 "Conn_Coaxial" H 14249 2435 50  0000 L CNN
+F 2 "Connector_Coaxial:SMB_Jack_Vertical" H 14150 2550 50  0001 C CNN
+F 3 " ~" H 14150 2550 50  0001 C CNN
+	1    14150 2550
+	1    0    0    -1
+$EndComp
+$Comp
+L Connector:Conn_Coaxial J1
+U 1 1 5BD270F6
+P 14050 3300
+F 0 "J1" H 14149 3276 50  0000 L CNN
+F 1 "Conn_Coaxial" H 14149 3185 50  0000 L CNN
+F 2 "Connector_Coaxial:SMB_Jack_Vertical" H 14050 3300 50  0001 C CNN
+F 3 " ~" H 14050 3300 50  0001 C CNN
+	1    14050 3300
+	1    0    0    -1
+$EndComp
+$Comp
+L RF_Switch:SA630D U2
+U 1 1 5BD29062
+P 12500 2150
+F 0 "U2" H 12575 2575 50  0000 C CNN
+F 1 "SA630D" H 12575 2484 50  0000 C CNN
+F 2 "Package_SO:SOIC-8_3.9x4.9mm_P1.27mm" H 12650 2600 50  0001 C CNN
+F 3 "" H 12500 2250 50  0001 C CNN
+	1    12500 2150
+	1    0    0    -1
+$EndComp
+Wire Wire Line
+	12100 2050 11750 2050
+Wire Wire Line
+	11750 2050 11750 3300
+Wire Wire Line
+	11750 3300 13850 3300
+Wire Wire Line
+	13050 1950 13800 1950
+Wire Wire Line
+	13800 1950 13800 1700
+Wire Wire Line
+	13800 1700 14050 1700
+Wire Wire Line
+	13050 2150 13800 2150
+Wire Wire Line
+	13800 2150 13800 2550
+Wire Wire Line
+	13800 2550 13950 2550
+$Comp
+L Device:R_Pack04 RN1
+U 1 1 5BD2A0ED
+P 11350 1200
+F 0 "RN1" H 11538 1246 50  0000 L CNN
+F 1 "R_Pack04" H 11538 1155 50  0000 L CNN
+F 2 "Resistor_SMD:R_Array_Convex_4x1206" V 11625 1200 50  0001 C CNN
+F 3 "~" H 11350 1200 50  0001 C CNN
+	1    11350 1200
+	1    0    0    -1
+$EndComp
+$Comp
+L Device:R_Pack04 RN2
+U 1 1 5BD2A53F
+P 13350 1200
+F 0 "RN2" H 13538 1246 50  0000 L CNN
+F 1 "R_Pack04" H 13538 1155 50  0000 L CNN
+F 2 "Resistor_SMD:R_Array_Convex_4x1206" V 13625 1200 50  0001 C CNN
+F 3 "~" H 13350 1200 50  0001 C CNN
+	1    13350 1200
+	1    0    0    -1
+$EndComp
+$Comp
+L c_pack04:C_Pack04 CN?
+U 1 1 5BD32370
+P 14700 1050
+F 0 "CN?" H 14783 966 50  0000 L CNN
+F 1 "C_Pack04" H 14783 875 50  0000 L CNN
+F 2 "" V 14870 920 50  0001 C CNN
+F 3 "~" H 14590 935 50  0001 C CNN
+	1    14700 1050
 	1    0    0    -1
 $EndComp

Commit message: minor changes - still experimenting
Parts:
- CN1: renamed from CN?; footprint (none) -> symbols:C_Array_Convex_4x1206
Changed lines of the file:
@@
 $EndComp
 $Comp
-L c_pack04:C_Pack04 CN?
+L c_pack04:C_Pack04 CN1
 U 1 1 5BD32370
 P 14700 1050
-F 0 "CN?" H 14783 966 50  0000 L CNN
+F 0 "CN1" H 14783 966 50  0000 L CNN
 F 1 "C_Pack04" H 14783 875 50  0000 L CNN
-F 2 "" V 14870 920 50  0001 C CNN
+F 2 "symbols:C_Array_Convex_4x1206" V 14870 920 50  0001 C CNN
 F 3 "~" H 14590 935 50  0001 C CNN
 	1    14700 1050

Commit message: pcb outline and start trim of connectors
Parts:
- CN9: footprint Connector_IDC:IDC-Header_2x15_P2.54mm_Vertical -> symbols:IDC-Pins_2x15_P2.54mm_Vertical
- U1: footprint Module:ST_Morpho_Connector_144_STLink -> symbols:ST_Nucleo_144_Large_Daughter
Changed lines of the file:
@@
 F 0 "U1" H 6900 9036 50  0000 C CNN
 F 1 "NUCLEO144-F746ZG" H 6900 9127 50  0000 C CNN
-F 2 "Module:ST_Morpho_Connector_144_STLink" H 7750 1500 50  0001 L CNN
+F 2 "symbols:ST_Nucleo_144_Large_Daughter" H 7750 1500 50  0001 L CNN
 F 3 "http://www.st.com/content/ccc/resource/technical/document/data_brief/group0/7b/df/1d/e9/64/55/43/8d/DM00247910/files/DM00247910.pdf/jcr:content/translations/en.DM00247910.pdf" H 6000 5450 50  0001 C CNN
 	1    6900 5150
@@
 F 0 "CN9" H 3006 8628 50  0000 C CNN
 F 1 "Conn_01x30_Male" H 3006 8537 50  0000 C CNN
-F 2 "Connector_IDC:IDC-Header_2x15_P2.54mm_Vertical" H 2900 7050 50  0001 C CNN
+F 2 "symbols:IDC-Pins_2x15_P2.54mm_Vertical" H 2900 7050 50  0001 C CNN
 F 3 "~" H 2900 7050 50  0001 C CNN
 	1    2900 7050

Commit message: Getting ready for proper start to project
Parts:
- removed CN1: C_Pack04, symbols:C_Array_Convex_4x1206, symbol c_pack04:C_Pack04
- removed U2: SA630D, Package_SO:SOIC-8_3.9x4.9mm_P1.27mm, symbol RF_Switch:SA630D
- added CN1: C_Pack04-c_pack04, spatboard:C_Array_Convex_5x1206, symbol splatsyms:C_Pack04-c_pack04
- added U2: SA630D-RF_Switch, Package_SO:SOIC-8_3.9x4.9mm_P1.27mm, symbol splatsyms:SA630D-RF_Switch
- CN10: footprint Connector_IDC:IDC-Header_2x17_P2.54mm_Vertical -> spatboard:IDC-Pins_2x17_P2.54mm_Vertical
- CN7: footprint Connector_IDC:IDC-Header_2x10_P2.54mm_Vertical -> spatboard:IDC-Pins_2x10_P2.54mm_Vertical
- CN8: footprint Connector_IDC:IDC-Header_2x08_P2.54mm_Vertical -> spatboard:IDC-Pins_2x8_P2.54mm_Vertical
Other:
- moved on the sheet: CN10, CN7, CN8
Changed lines of the file:
@@
 L Connector:Conn_01x34_Male CN10
 U 1 1 5BD04B56
-P 10150 7350
-F 0 "CN10" H 10256 9128 50  0000 C CNN
-F 1 "Conn_01x34_Male" H 10256 9037 50  0000 C CNN
-F 2 "Connector_IDC:IDC-Header_2x17_P2.54mm_Vertical" H 10150 7350 50  0001 C CNN
-F 3 "~" H 10150 7350 50  0001 C CNN
-	1    10150 7350
+P 9950 6350
+F 0 "CN10" H 10056 8128 50  0000 C CNN
+F 1 "Conn_01x34_Male" H 10056 8037 50  0000 C CNN
+F 2 "spatboard:IDC-Pins_2x17_P2.54mm_Vertical" H 9950 6350 50  0001 C CNN
+F 3 "~" H 9950 6350 50  0001 C CNN
+	1    9950 6350
 	1    0    0    -1
 $EndComp
@@
 L Connector:Conn_01x20_Male CN7
 U 1 1 5BD04C2E
-P 10100 2850
-F 0 "CN7" H 10206 3928 50  0000 C CNN
-F 1 "Conn_01x20_Male" H 10206 3837 50  0000 C CNN
-F 2 "Connector_IDC:IDC-Header_2x10_P2.54mm_Vertical" H 10100 2850 50  0001 C CNN
-F 3 "~" H 10100 2850 50  0001 C CNN
-	1    10100 2850
+P 9450 2900
+F 0 "CN7" H 9556 3978 50  0000 C CNN
+F 1 "Conn_01x20_Male" H 9556 3887 50  0000 C CNN
+F 2 "spatboard:IDC-Pins_2x10_P2.54mm_Vertical" H 9450 2900 50  0001 C CNN
+F 3 "~" H 9450 2900 50  0001 C CNN
+	1    9450 2900
 	1    0    0    -1
 $EndComp
@@
 L Connector:Conn_01x16_Male CN8
 U 1 1 5BD04E48
-P 2650 3350
-F 0 "CN8" H 2756 4228 50  0000 C CNN
-F 1 "Conn_01x16_Male" H 2756 4137 50  0000 C CNN
-F 2 "Connector_IDC:IDC-Header_2x08_P2.54mm_Vertical" H 2650 3350 50  0001 C CNN
-F 3 "~" H 2650 3350 50  0001 C CNN
-	1    2650 3350
+P 2900 3300
+F 0 "CN8" H 3006 4178 50  0000 C CNN
+F 1 "Conn_01x16_Male" H 3006 4087 50  0000 C CNN
+F 2 "spatboard:IDC-Pins_2x8_P2.54mm_Vertical" H 2900 3300 50  0001 C CNN
+F 3 "~" H 2900 3300 50  0001 C CNN
+	1    2900 3300
 	1    0    0    -1
 $EndComp
@@
 F 3 " ~" H 14050 3300 50  0001 C CNN
 	1    14050 3300
-	1    0    0    -1
-$EndComp
-$Comp
-L RF_Switch:SA630D U2
-U 1 1 5BD29062
-P 12500 2150
-F 0 "U2" H 12575 2575 50  0000 C CNN
-F 1 "SA630D" H 12575 2484 50  0000 C CNN
-F 2 "Package_SO:SOIC-8_3.9x4.9mm_P1.27mm" H 12650 2600 50  0001 C CNN
-F 3 "" H 12500 2250 50  0001 C CNN
-	1    12500 2150
 	1    0    0    -1
 $EndComp
@@
 $EndComp
 $Comp
-L c_pack04:C_Pack04 CN1
-U 1 1 5BD32370
-P 14700 1050
-F 0 "CN1" H 14783 966 50  0000 L CNN
-F 1 "C_Pack04" H 14783 875 50  0000 L CNN
-F 2 "symbols:C_Array_Convex_4x1206" V 14870 920 50  0001 C CNN
-F 3 "~" H 14590 935 50  0001 C CNN
-	1    14700 1050
+L splatsyms:SA630D-RF_Switch U2
+U 1 1 5BD7BF76
+P 12500 2150
+F 0 "U2" H 12575 2575 50  0000 C CNN
+F 1 "SA630D-RF_Switch" H 12575 2484 50  0000 C CNN
+F 2 "Package_SO:SOIC-8_3.9x4.9mm_P1.27mm" H 12650 2600 50  0001 C CNN
+F 3 "" H 12500 2250 50  0001 C CNN
+	1    12500 2150
 	1    0    0    -1
 $EndComp
+$Comp
+L splatsyms:C_Pack04-c_pack04 CN1
+U 1 1 5BD7C218
+P 13850 3700
+F 0 "CN1" H 13933 3616 50  0000 L CNN
+F 1 "C_Pack04-c_pack04" H 13933 3525 50  0000 L CNN
+F 2 "spatboard:C_Array_Convex_5x1206" V 14020 3570 50  0001 C CNN
+F 3 "" H 13740 3585 50  0001 C CNN
+	1    13850 3700
+	1    0    0    -1
+$EndComp

Commit message: Cropped PCB to clear STM board buttons
Added GPS module connector and silkscreen
Parts:
- added U3: MCP6S93-X_UN, MSOP10_MC, symbol splatsyms:MCP6S93-X_UN
- added U4: ublox_chinese_PCB_module, Blox_Neo7module, symbol splatsyms:ublox_SAM-M8Q
- CN1: value C_Pack04-c_pack04 -> C_Pack04; footprint spatboard:C_Array_Convex_5x1206 -> (none)
- CN10: footprint spatboard:IDC-Pins_2x17_P2.54mm_Vertical -> (none)
- CN7: footprint spatboard:IDC-Pins_2x10_P2.54mm_Vertical -> (none)
- CN8: footprint spatboard:IDC-Pins_2x8_P2.54mm_Vertical -> (none)
- CN9: footprint symbols:IDC-Pins_2x15_P2.54mm_Vertical -> (none)
- J1, J2, J3: footprint Connector_Coaxial:SMB_Jack_Vertical -> (none)
- RN1, RN2: footprint Resistor_SMD:R_Array_Convex_4x1206 -> (none)
- U1: footprint symbols:ST_Nucleo_144_Large_Daughter -> Module:ST_Morpho_Connector_144_STLink
Connections:
- wire segments 9 -> 12
Other:
- moved on the sheet: CN1, CN9
Changed lines of the file:
@@
 F 0 "U1" H 6900 9036 50  0000 C CNN
 F 1 "NUCLEO144-F746ZG" H 6900 9127 50  0000 C CNN
-F 2 "symbols:ST_Nucleo_144_Large_Daughter" H 7750 1500 50  0001 L CNN
-F 3 "http://www.st.com/content/ccc/resource/technical/document/data_brief/group0/7b/df/1d/e9/64/55/43/8d/DM00247910/files/DM00247910.pdf/jcr:content/translations/en.DM00247910.pdf" H 6000 5450 50  0001 C CNN
+F 2 "Module:ST_Morpho_Connector_144_STLink" H 7750 1500 50  0001 L CNN
+F 3 "" H 6000 5450 50  0001 C CNN
 	1    6900 5150
 	-1   0    0    1
@@
 F 0 "CN10" H 10056 8128 50  0000 C CNN
 F 1 "Conn_01x34_Male" H 10056 8037 50  0000 C CNN
-F 2 "spatboard:IDC-Pins_2x17_P2.54mm_Vertical" H 9950 6350 50  0001 C CNN
-F 3 "~" H 9950 6350 50  0001 C CNN
+F 2 "" H 9950 6350 50  0001 C CNN
+F 3 "" H 9950 6350 50  0001 C CNN
 	1    9950 6350
 	1    0    0    -1
@@
 F 0 "CN7" H 9556 3978 50  0000 C CNN
 F 1 "Conn_01x20_Male" H 9556 3887 50  0000 C CNN
-F 2 "spatboard:IDC-Pins_2x10_P2.54mm_Vertical" H 9450 2900 50  0001 C CNN
-F 3 "~" H 9450 2900 50  0001 C CNN
+F 2 "" H 9450 2900 50  0001 C CNN
+F 3 "" H 9450 2900 50  0001 C CNN
 	1    9450 2900
 	1    0    0    -1
@@
 L Connector:Conn_01x30_Male CN9
 U 1 1 5BD04D97
-P 2900 7050
-F 0 "CN9" H 3006 8628 50  0000 C CNN
-F 1 "Conn_01x30_Male" H 3006 8537 50  0000 C CNN
-F 2 "symbols:IDC-Pins_2x15_P2.54mm_Vertical" H 2900 7050 50  0001 C CNN
-F 3 "~" H 2900 7050 50  0001 C CNN
-	1    2900 7050
+P 3150 6500
+F 0 "CN9" H 3256 8078 50  0000 C CNN
+F 1 "Conn_01x30_Male" H 3256 7987 50  0000 C CNN
+F 2 "" H 3150 6500 50  0001 C CNN
+F 3 "" H 3150 6500 50  0001 C CNN
+	1    3150 6500
 	1    0    0    -1
 $EndComp
@@
 F 0 "CN8" H 3006 4178 50  0000 C CNN
 F 1 "Conn_01x16_Male" H 3006 4087 50  0000 C CNN
-F 2 "spatboard:IDC-Pins_2x8_P2.54mm_Vertical" H 2900 3300 50  0001 C CNN
-F 3 "~" H 2900 3300 50  0001 C CNN
+F 2 "" H 2900 3300 50  0001 C CNN
+F 3 "" H 2900 3300 50  0001 C CNN
 	1    2900 3300
 	1    0    0    -1
@@
 F 0 "J3" H 14349 1676 50  0000 L CNN
 F 1 "Conn_Coaxial" H 14349 1585 50  0000 L CNN
-F 2 "Connector_Coaxial:SMB_Jack_Vertical" H 14250 1700 50  0001 C CNN
-F 3 " ~" H 14250 1700 50  0001 C CNN
+F 2 "" H 14250 1700 50  0001 C CNN
+F 3 "" H 14250 1700 50  0001 C CNN
 	1    14250 1700
 	1    0    0    -1
@@
 F 0 "J2" H 14249 2526 50  0000 L CNN
 F 1 "Conn_Coaxial" H 14249 2435 50  0000 L CNN
-F 2 "Connector_Coaxial:SMB_Jack_Vertical" H 14150 2550 50  0001 C CNN
-F 3 " ~" H 14150 2550 50  0001 C CNN
+F 2 "" H 14150 2550 50  0001 C CNN
+F 3 "" H 14150 2550 50  0001 C CNN
 	1    14150 2550
 	1    0    0    -1
@@
 F 0 "J1" H 14149 3276 50  0000 L CNN
 F 1 "Conn_Coaxial" H 14149 3185 50  0000 L CNN
-F 2 "Connector_Coaxial:SMB_Jack_Vertical" H 14050 3300 50  0001 C CNN
-F 3 " ~" H 14050 3300 50  0001 C CNN
+F 2 "" H 14050 3300 50  0001 C CNN
+F 3 "" H 14050 3300 50  0001 C CNN
 	1    14050 3300
 	1    0    0    -1
@@
 F 0 "RN1" H 11538 1246 50  0000 L CNN
 F 1 "R_Pack04" H 11538 1155 50  0000 L CNN
-F 2 "Resistor_SMD:R_Array_Convex_4x1206" V 11625 1200 50  0001 C CNN
-F 3 "~" H 11350 1200 50  0001 C CNN
+F 2 "" V 11625 1200 50  0001 C CNN
+F 3 "" H 11350 1200 50  0001 C CNN
 	1    11350 1200
 	1    0    0    -1
@@
 F 0 "RN2" H 13538 1246 50  0000 L CNN
 F 1 "R_Pack04" H 13538 1155 50  0000 L CNN
-F 2 "Resistor_SMD:R_Array_Convex_4x1206" V 13625 1200 50  0001 C CNN
-F 3 "~" H 13350 1200 50  0001 C CNN
+F 2 "" V 13625 1200 50  0001 C CNN
+F 3 "" H 13350 1200 50  0001 C CNN
 	1    13350 1200
 	1    0    0    -1
@@
 L splatsyms:C_Pack04-c_pack04 CN1
 U 1 1 5BD7C218
-P 13850 3700
-F 0 "CN1" H 13933 3616 50  0000 L CNN
-F 1 "C_Pack04-c_pack04" H 13933 3525 50  0000 L CNN
-F 2 "spatboard:C_Array_Convex_5x1206" V 14020 3570 50  0001 C CNN
-F 3 "" H 13740 3585 50  0001 C CNN
-	1    13850 3700
+P 13600 3900
+F 0 "CN1" H 13683 3816 50  0000 L CNN
+F 1 "C_Pack04" H 13683 3725 50  0000 L CNN
+F 2 "" V 13770 3770 50  0001 C CNN
+F 3 "" H 13490 3785 50  0001 C CNN
+	1    13600 3900
 	1    0    0    -1
 $EndComp
+$Comp
+L splatsyms:MCP6S93-X_UN U3
+U 1 1 5BD7F0EC
+P 11600 5200
+F 0 "U3" H 12400 5587 60  0000 C CNN
+F 1 "MCP6S93-X_UN" H 12400 5481 60  0000 C CNN
+F 2 "MSOP10_MC" H 12400 5440 60  0001 C CNN
+F 3 "" H 11600 5200 60  0000 C CNN
+	1    11600 5200
+	1    0    0    -1
+$EndComp
+Wire Wire Line
+	14050 3500 11000 3500
+Wire Wire Line
+	11000 3500 11000 5600
+Wire Wire Line
+	11000 5600 11600 5600
+$Comp
+L splatsyms:ublox_SAM-M8Q U4
+U 1 1 5BD908A5
+P 13650 7150
+F 0 "U4" H 13650 7828 50  0000 C CNN
+F 1 "ublox_chinese_PCB_module" H 13650 7737 50  0000 C CNN
+F 2 "Blox_Neo7module" H 13650 7050 50  0001 C CNN
+F 3 "" H 13650 7150 50  0001 C CNN
+F 4 "M20-7890546" H 13650 7150 50  0001 C CNN "RS Components"
+	1    13650 7150
+	1    0    0    -1
+$EndComp

Commit message: Footprints re-assigned
PCB had lost associations
Parts:
- CN1: footprint (none) -> spatboard:C_Array_Convex_4x1206
- CN10: footprint (none) -> spatboard:IDC-Pins_2x17_P2.54mm_Vertical
- CN7: footprint (none) -> spatboard:IDC-Pins_2x10_P2.54mm_Vertical
- CN8: footprint (none) -> spatboard:IDC-Pins_2x8_P2.54mm_Vertical
- CN9: footprint (none) -> spatboard:IDC-Pins_2x15_P2.54mm_Vertical
- J1, J2, J3: footprint (none) -> Connector_Coaxial:SMA_Amphenol_132134-11_Vertical
- RN1, RN2: footprint (none) -> Resistor_SMD:R_Array_Convex_4x1206
- U1: footprint Module:ST_Morpho_Connector_144_STLink -> spatboard:ST_Nucleo_144_Large_Daughter
- U3: footprint MSOP10_MC -> Package_SO:MSOP-10_3x3mm_P0.5mm
- U4: footprint Blox_Neo7module -> spatboard:GPS_IDC-Header_2x05_P2.54mm_Horizontal
Connections:
- net labels added: +3V3, +5V, GND, IOREF, PC10, PC11, PC12, PC8, PC9, PD2, PG2, PG3, RESET, VIN
- wire segments 12 -> 13
Other:
- moved on the sheet: CN10, CN7, CN8, CN9, J1, U3
Changed lines of the file:
@@
 F 0 "U1" H 6900 9036 50  0000 C CNN
 F 1 "NUCLEO144-F746ZG" H 6900 9127 50  0000 C CNN
-F 2 "Module:ST_Morpho_Connector_144_STLink" H 7750 1500 50  0001 L CNN
+F 2 "spatboard:ST_Nucleo_144_Large_Daughter" H 7750 1500 50  0001 L CNN
 F 3 "" H 6000 5450 50  0001 C CNN
 	1    6900 5150
@@
 L Connector:Conn_01x34_Male CN10
 U 1 1 5BD04B56
-P 9950 6350
-F 0 "CN10" H 10056 8128 50  0000 C CNN
-F 1 "Conn_01x34_Male" H 10056 8037 50  0000 C CNN
-F 2 "" H 9950 6350 50  0001 C CNN
-F 3 "" H 9950 6350 50  0001 C CNN
-	1    9950 6350
+P 9900 6150
+F 0 "CN10" H 10006 7928 50  0000 C CNN
+F 1 "Conn_01x34_Male" H 10006 7837 50  0000 C CNN
+F 2 "spatboard:IDC-Pins_2x17_P2.54mm_Vertical" H 9900 6150 50  0001 C CNN
+F 3 "" H 9900 6150 50  0001 C CNN
+	1    9900 6150
 	1    0    0    -1
 $EndComp
@@
 L Connector:Conn_01x20_Male CN7
 U 1 1 5BD04C2E
-P 9450 2900
-F 0 "CN7" H 9556 3978 50  0000 C CNN
-F 1 "Conn_01x20_Male" H 9556 3887 50  0000 C CNN
-F 2 "" H 9450 2900 50  0001 C CNN
-F 3 "" H 9450 2900 50  0001 C CNN
-	1    9450 2900
+P 9500 2800
+F 0 "CN7" H 9606 3878 50  0000 C CNN
+F 1 "Conn_01x20_Male" H 9606 3787 50  0000 C CNN
+F 2 "spatboard:IDC-Pins_2x10_P2.54mm_Vertical" H 9500 2800 50  0001 C CNN
+F 3 "" H 9500 2800 50  0001 C CNN
+	1    9500 2800
 	1    0    0    -1
 $EndComp
@@
 L Connector:Conn_01x30_Male CN9
 U 1 1 5BD04D97
-P 3150 6500
-F 0 "CN9" H 3256 8078 50  0000 C CNN
-F 1 "Conn_01x30_Male" H 3256 7987 50  0000 C CNN
-F 2 "" H 3150 6500 50  0001 C CNN
-F 3 "" H 3150 6500 50  0001 C CNN
-	1    3150 6500
+P 3150 6600
+F 0 "CN9" H 3256 8178 50  0000 C CNN
+F 1 "Conn_01x30_Male" H 3256 8087 50  0000 C CNN
+F 2 "spatboard:IDC-Pins_2x15_P2.54mm_Vertical" H 3150 6600 50  0001 C CNN
+F 3 "" H 3150 6600 50  0001 C CNN
+	1    3150 6600
 	1    0    0    -1
 $EndComp
@@
 L Connector:Conn_01x16_Male CN8
 U 1 1 5BD04E48
-P 2900 3300
-F 0 "CN8" H 3006 4178 50  0000 C CNN
-F 1 "Conn_01x16_Male" H 3006 4087 50  0000 C CNN
-F 2 "" H 2900 3300 50  0001 C CNN
-F 3 "" H 2900 3300 50  0001 C CNN
-	1    2900 3300
+P 2950 3150
+F 0 "CN8" H 3056 4028 50  0000 C CNN
+F 1 "Conn_01x16_Male" H 3056 3937 50  0000 C CNN
+F 2 "spatboard:IDC-Pins_2x8_P2.54mm_Vertical" H 2950 3150 50  0001 C CNN
+F 3 "" H 2950 3150 50  0001 C CNN
+	1    2950 3150
 	1    0    0    -1
 $EndComp
@@
 F 0 "J3" H 14349 1676 50  0000 L CNN
 F 1 "Conn_Coaxial" H 14349 1585 50  0000 L CNN
-F 2 "" H 14250 1700 50  0001 C CNN
+F 2 "Connector_Coaxial:SMA_Amphenol_132134-11_Vertical" H 14250 1700 50  0001 C CNN
 F 3 "" H 14250 1700 50  0001 C CNN
 	1    14250 1700
@@
 F 0 "J2" H 14249 2526 50  0000 L CNN
 F 1 "Conn_Coaxial" H 14249 2435 50  0000 L CNN
-F 2 "" H 14150 2550 50  0001 C CNN
+F 2 "Connector_Coaxial:SMA_Amphenol_132134-11_Vertical" H 14150 2550 50  0001 C CNN
 F 3 "" H 14150 2550 50  0001 C CNN
 	1    14150 2550
@@
 L Connector:Conn_Coaxial J1
 U 1 1 5BD270F6
-P 14050 3300
-F 0 "J1" H 14149 3276 50  0000 L CNN
-F 1 "Conn_Coaxial" H 14149 3185 50  0000 L CNN
-F 2 "" H 14050 3300 50  0001 C CNN
-F 3 "" H 14050 3300 50  0001 C CNN
-	1    14050 3300
+P 14050 3200
+F 0 "J1" H 14149 3176 50  0000 L CNN
+F 1 "Conn_Coaxial" H 14149 3085 50  0000 L CNN
+F 2 "Connector_Coaxial:SMA_Amphenol_132134-11_Vertical" H 14050 3200 50  0001 C CNN
+F 3 "" H 14050 3200 50  0001 C CNN
+	1    14050 3200
 	1    0    0    -1
 $EndComp
@@
 	12100 2050 11750 2050
 Wire Wire Line
-	11750 2050 11750 3300
-Wire Wire Line
-	11750 3300 13850 3300
+	11750 2050 11750 3200
+Wire Wire Line
+	11750 3200 13850 3200
 Wire Wire Line
 	13050 1950 13800 1950
@@
 F 0 "RN1" H 11538 1246 50  0000 L CNN
 F 1 "R_Pack04" H 11538 1155 50  0000 L CNN
-F 2 "" V 11625 1200 50  0001 C CNN
+F 2 "Resistor_SMD:R_Array_Convex_4x1206" V 11625 1200 50  0001 C CNN
 F 3 "" H 11350 1200 50  0001 C CNN
 	1    11350 1200
@@
 F 0 "RN2" H 13538 1246 50  0000 L CNN
 F 1 "R_Pack04" H 13538 1155 50  0000 L CNN
-F 2 "" V 13625 1200 50  0001 C CNN
+F 2 "Resistor_SMD:R_Array_Convex_4x1206" V 13625 1200 50  0001 C CNN
 F 3 "" H 13350 1200 50  0001 C CNN
 	1    13350 1200
@@
 F 0 "CN1" H 13683 3816 50  0000 L CNN
 F 1 "C_Pack04" H 13683 3725 50  0000 L CNN
-F 2 "" V 13770 3770 50  0001 C CNN
+F 2 "spatboard:C_Array_Convex_4x1206" V 13770 3770 50  0001 C CNN
 F 3 "" H 13490 3785 50  0001 C CNN
 	1    13600 3900
@@
 L splatsyms:MCP6S93-X_UN U3
 U 1 1 5BD7F0EC
-P 11600 5200
-F 0 "U3" H 12400 5587 60  0000 C CNN
-F 1 "MCP6S93-X_UN" H 12400 5481 60  0000 C CNN
-F 2 "MSOP10_MC" H 12400 5440 60  0001 C CNN
-F 3 "" H 11600 5200 60  0000 C CNN
-	1    11600 5200
+P 12800 5000
+F 0 "U3" H 13600 5387 60  0000 C CNN
+F 1 "MCP6S93-X_UN" H 13600 5281 60  0000 C CNN
+F 2 "Package_SO:MSOP-10_3x3mm_P0.5mm" H 13600 5240 60  0001 C CNN
+F 3 "" H 12800 5000 60  0000 C CNN
+	1    12800 5000
 	1    0    0    -1
 $EndComp
@@
 	11000 3500 11000 5600
 Wire Wire Line
-	11000 5600 11600 5600
+	13350 6550 13950 6550
 $Comp
 L splatsyms:ublox_SAM-M8Q U4
 U 1 1 5BD908A5
-P 13650 7150
-F 0 "U4" H 13650 7828 50  0000 C CNN
-F 1 "ublox_chinese_PCB_module" H 13650 7737 50  0000 C CNN
-F 2 "Blox_Neo7module" H 13650 7050 50  0001 C CNN
-F 3 "" H 13650 7150 50  0001 C CNN
-F 4 "M20-7890546" H 13650 7150 50  0001 C CNN "RS Components"
-	1    13650 7150
-	1    0    0    -1
-$EndComp
+P 13050 6550
+F 0 "U4" H 13050 7228 50  0000 C CNN
+F 1 "ublox_chinese_PCB_module" H 13050 7137 50  0000 C CNN
+F 2 "spatboard:GPS_IDC-Header_2x05_P2.54mm_Horizontal" H 13050 6450 50  0001 C CNN
+F 3 "" H 13050 6550 50  0001 C CNN
+F 4 "M20-7890546" H 13050 6550 50  0001 C CNN "RS Components"
+	1    13050 6550
+	1    0    0    -1
+$EndComp
+Text HLabel 3150 2550 2    50   Input ~ 0
+PC8
+Text HLabel 3150 2750 2    50   Input ~ 0
+PC9
+Text HLabel 3150 2650 2    50   Input ~ 0
+IOREF
+Text HLabel 3150 2850 2    50   Input ~ 0
+RESET
+Text HLabel 3150 2950 2    50   Input ~ 0
+PC10
+Text HLabel 3150 3050 2    50   Input ~ 0
++3V3
+Text HLabel 3150 3150 2    50   Input ~ 0
+PC11
+Text HLabel 3150 3250 2    50   Input ~ 0
++5V
+Text HLabel 3150 3350 2    50   Input ~ 0
+PC12
+Text HLabel 3150 3450 2    50   Input ~ 0
+GND
+Text HLabel 3150 3550 2    50   Input ~ 0
+PD2
+Text HLabel 3200 3650 2    50   Input ~ 0
+GND
+Text HLabel 3150 3750 2    50   Input ~ 0
+PG2
+Text HLabel 3150 3850 2    50   Input ~ 0
+VIN
+Text HLabel 3150 3950 2    50   Input ~ 0
+PG3
+Connection ~ 11750 3200
+Wire Wire Line
+	11750 3200 11750 3300
 $EndSCHEMATC
