File: stmsplat1.sch (KiCad schematic (older format))
At the start: 14 parts, among them CN1 C_Pack04, CN10 Conn_01x34_Male, CN7 Conn_01x20_Male, CN8 Conn_01x16_Male, CN9 Conn_01x30_Male, J1 Conn_Coaxial, J2 Conn_Coaxial, J3 Conn_Coaxial, U1 NUCLEO144-F746ZG, U2 SA630D-RF_Switch, U3 MCP6S93-X_UN, U4 ublox_chinese_PCB_module

Commit message: Added Arduino Header Labels
Connections:
- net labels added: AGND, AVDD, PA0, PA15, PA3, PA4, PA5, PA6, PA7, PB0, PB1, PB10, PB11, PB12, PB13, PB15, PB2, PB3, PB4, PB5, PB6, PB8, PB9, PC0, PC2, PC3, PC6, PC7, PD0, PD1, PD11, PD12, PD13, PD14, PD15, PD3, PD4, PD5, PD6, PD7, PE0, PE10, PE11, PE12, PE13, PE14, PE15, PE2, PE3, PE4, PE5, PE6, PE7, PE8, PE9, PF0, PF1, PF10, PF12, PF13, PF14, PF15, PF2, PF3, PF4, PF5, PF7, PF8, PF9, PG0, PG1, PG14, PG9
Changed lines of the file:
@@
 Wire Wire Line
 	11750 3200 11750 3300
+Text HLabel 3350 5200 2    50   Input ~ 0
+PA3
+Text HLabel 3350 5300 2    50   Input ~ 0
+PD7
+Text HLabel 3350 5400 2    50   Input ~ 0
+PC0
+Text HLabel 3350 5500 2    50   Input ~ 0
+PD6
+Text HLabel 3350 5600 2    50   Input ~ 0
+PC3
+Text HLabel 3350 5700 2    50   Input ~ 0
+PD5
+Text HLabel 3350 5800 2    50   Input ~ 0
+PF3
+Text HLabel 3350 5900 2    50   Input ~ 0
+PD4
+Text HLabel 3350 6000 2    50   Input ~ 0
+PF5
+Text HLabel 3350 6100 2    50   Input ~ 0
+PD3
+Text HLabel 3350 6200 2    50   Input ~ 0
+PF10
+Text HLabel 3350 6300 2    50   Input ~ 0
+GND
+Text HLabel 3350 6500 2    50   Input ~ 0
+PE2
+Text HLabel 3350 6600 2    50   Input ~ 0
+PA7
+Text HLabel 3350 6700 2    50   Input ~ 0
+PE4
+Text HLabel 3350 6800 2    50   Input ~ 0
+PF2
+Text HLabel 3350 6900 2    50   Input ~ 0
+PE5
+Text HLabel 3350 7000 2    50   Input ~ 0
+PF1
+Text HLabel 3350 7100 2    50   Input ~ 0
+PE6
+Text HLabel 3350 7200 2    50   Input ~ 0
+PF0
+Text HLabel 3350 7300 2    50   Input ~ 0
+PE3
+Text HLabel 3350 7400 2    50   Input ~ 0
+GND
+Text HLabel 3350 7500 2    50   Input ~ 0
+PF8
+Text HLabel 3350 7600 2    50   Input ~ 0
+PD0
+Text HLabel 3350 7700 2    50   Input ~ 0
+PF7
+Text HLabel 3350 7800 2    50   Input ~ 0
+PD1
+Text HLabel 3350 7900 2    50   Input ~ 0
+PF9
+Text HLabel 3350 8000 2    50   Input ~ 0
+PG0
+Text HLabel 3350 8100 2    50   Input ~ 0
+PG1
+Text HLabel 10100 4550 2    50   Input ~ 0
+AVDD
+Text HLabel 10100 4650 2    50   Input ~ 0
+PF13
+Text HLabel 10100 4750 2    50   Input ~ 0
+AGND
+Text HLabel 10100 4850 2    50   Input ~ 0
+PE9
+Text HLabel 10100 4950 2    50   Input ~ 0
+GND
+Text HLabel 10100 5050 2    50   Input ~ 0
+PE11
+Text HLabel 10100 5150 2    50   Input ~ 0
+PB1
+Text HLabel 10100 5250 2    50   Input ~ 0
+PF14
+Text HLabel 10100 5350 2    50   Input ~ 0
+PC2
+Text HLabel 10100 5450 2    50   Input ~ 0
+PE13
+Text HLabel 10100 5550 2    50   Input ~ 0
+PF4
+Text HLabel 10100 5650 2    50   Input ~ 0
+PF15
+Text HLabel 10100 5750 2    50   Input ~ 0
+PB6
+Text HLabel 10100 5850 2    50   Input ~ 0
+PG14
+Text HLabel 10100 5950 2    50   Input ~ 0
+PB2
+Text HLabel 10100 6050 2    50   Input ~ 0
+PG9
+Text HLabel 10100 6150 2    50   Input ~ 0
+GND
+Text HLabel 10100 6250 2    50   Input ~ 0
+PE8
+Text HLabel 10100 6350 2    50   Input ~ 0
+PD13
+Text HLabel 10100 6450 2    50   Input ~ 0
+PE7
+Text HLabel 10100 6550 2    50   Input ~ 0
+PD12
+Text HLabel 10100 6650 2    50   Input ~ 0
+GND
+Text HLabel 10100 6750 2    50   Input ~ 0
+PD11
+Text HLabel 10100 6850 2    50   Input ~ 0
+PE10
+Text HLabel 10100 6950 2    50   Input ~ 0
+PE2
+Text HLabel 10100 7050 2    50   Input ~ 0
+PE12
+Text HLabel 10100 7150 2    50   Input ~ 0
+GND
+Text HLabel 10100 7250 2    50   Input ~ 0
+PE14
+Text HLabel 10100 7350 2    50   Input ~ 0
+PA0
+Text HLabel 10100 7450 2    50   Input ~ 0
+PE15
+Text HLabel 10100 7550 2    50   Input ~ 0
+PB0
+Text HLabel 10100 7650 2    50   Input ~ 0
+PB10
+Text HLabel 10100 7750 2    50   Input ~ 0
+PE0
+Text HLabel 10100 7850 2    50   Input ~ 0
+PB11
+Text HLabel 9700 1900 2    50   Input ~ 0
+PC6
+Text HLabel 9700 2000 2    50   Input ~ 0
+PB8
+Text HLabel 9700 2100 2    50   Input ~ 0
+PB15
+Text HLabel 9700 2200 2    50   Input ~ 0
+PB9
+Text HLabel 9700 2300 2    50   Input ~ 0
+PB13
+Text HLabel 9700 2400 2    50   Input ~ 0
+AVDD
+Text HLabel 9700 2500 2    50   Input ~ 0
+PB12
+Text HLabel 9700 2600 2    50   Input ~ 0
+GND
+Text HLabel 9700 2700 2    50   Input ~ 0
+PA15
+Text HLabel 9700 2800 2    50   Input ~ 0
+PA5
+Text HLabel 9700 2900 2    50   Input ~ 0
+PC7
+Text HLabel 9700 3000 2    50   Input ~ 0
+PA6
+Text HLabel 9700 3100 2    50   Input ~ 0
+PB5
+Text HLabel 9700 3200 2    50   Input ~ 0
+PA7
+Text HLabel 9700 3300 2    50   Input ~ 0
+PB3
+Text HLabel 9700 3400 2    50   Input ~ 0
+PD14
+Text HLabel 9700 3500 2    50   Input ~ 0
+PA4
+Text HLabel 9700 3600 2    50   Input ~ 0
+PD15
+Text HLabel 9700 3700 2    50   Input ~ 0
+PB4
+Text HLabel 9700 3800 2    50   Input ~ 0
+PF12
 $EndSCHEMATC

Commit message: Added input lowpass filter
Parts:
- removed J1, J2: Conn_Coaxial, Connector_Coaxial:SMA_Amphenol_132134-11_Vertical, symbol Connector:Conn_Coaxial
- removed RN1, RN2: R_Pack04, Resistor_SMD:R_Array_Convex_4x1206, symbol Device:R_Pack04
- removed U2: SA630D-RF_Switch, Package_SO:SOIC-8_3.9x4.9mm_P1.27mm, symbol splatsyms:SA630D-RF_Switch
- added C1, C2: 1uF, Capacitor_THT:CP_Radial_D5.0mm_P2.50mm, symbol Device:CP
- added C3: 560pF, Capacitor_SMD:C_0805_2012Metric_Pad1.15x1.40mm_HandSolder, symbol Device:C
- added C4: 240pF, Capacitor_SMD:C_0805_2012Metric_Pad1.15x1.40mm_HandSolder, symbol Device:C
- added D1: SMAJ8.0CA Bourns 9V, Diode_SMD:D_SMA_Handsoldering, symbol Device:D_TVS
- added FB1, FB2: Ferrite_Bead, Inductor_SMD:L_0805_2012Metric, symbol Device:Ferrite_Bead
- added L1: 620nH, Inductor_SMD:L_1210_3225Metric_Pad1.42x2.65mm_HandSolder, symbol Device:L
- added L2: 1.5uH, Inductor_SMD:L_1210_3225Metric_Pad1.42x2.65mm_HandSolder, symbol Device:L
- added R1, R2: 100R, Resistor_SMD:R_2010_5025Metric_Pad1.52x2.65mm_HandSolder, symbol Device:R
- added RN3: 4K7, Resistor_SMD:R_Array_Convex_4x1206, symbol Device:R_Pack04
- added U2: AD8310, Package_SO:MSOP-8-1EP_3x3mm_P0.65mm_EP2.54x2.8mm, symbol splatsyms:AD8310
- added U5: Opamp_Quad_MCP6024, symbol Device:Opamp_Quad_Generic
- CN1: value C_Pack04 -> 10n; symbol splatsyms:C_Pack04-c_pack04 -> stmsplat1-rescue:C_Pack04-c_pack04-splatsyms
- U4: symbol splatsyms:ublox_SAM-M8Q -> stmsplat1-rescue:ublox_SAM-M8Q-splatsyms
Connections:
- net labels added: A3V3
- wire segments 13 -> 88
Other:
- moved on the sheet: CN1, CN10, CN7, CN8, CN9, J3, U1, U3
